File: 3D Model/3DModelProject/3DModelProject.kicad_pcb (KiCad board)
At the start: 4 copper layers, 105 x 49.2 mm, 12 parts, among them J1 Power, J2 USB_B_Micro, J3 Tire Sensor, J4 BMS Sensor, J5 CAN Connector, J6 SWD, U1 STM32F765ZITx, U2 SN65HVD255D, U3 ICM-20602, U4 LP5907MFX-3.3, U5 USB3341, U6 TPD2EUSB30A

Commit message: zips
Parts:
- added H1: MountingHole, MountingHole:MountingHole_2.5mm_Pad_TopBottom, F.Cu at (171.5, 92.0)
- added H2: MountingHole, MountingHole:MountingHole_2.5mm_Pad_TopBottom, F.Cu at (171.5, 43.5)
- added H3: MountingHole, MountingHole:MountingHole_2.5mm_Pad_TopBottom, F.Cu at (72.5, 92.0)
- added H4: MountingHole, MountingHole:MountingHole_2.5mm_Pad_TopBottom, F.Cu at (72.5, 43.5)
- moved J6 7.39 mm to (86.1, 50.5)
Routing:
- net /SWDIO: track 39.3 -> 38.6 mm
Other:
- board size 105 x 49.2 mm -> 105.1 x 54.7 mm
