File: 3D Model/3DModelProject/3DModelProject.kicad_sch (KiCad schematic)
At the start: 12 parts, among them J1 Power, J2 USB_B_Micro, J3 Tire Sensor, J4 BMS Sensor, J5 CAN Connector, J6 SWD, U1 STM32F765ZITx, U2 SN65HVD255D, U3 ICM-20602, U5 USB3341, U6 TPD2EUSB30A

Commit message: zips
Parts:
- added H1, H2, H3, H4: MountingHole, MountingHole:MountingHole_2.5mm_Pad_TopBottom, symbol Mechanical:MountingHole
- gave numbers to parts that had none: 1
Changed lines of the file:
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@@
     (pin "1")
+  )
+  (symbol (lib_id "Mechanical:MountingHole") (at 200.66 55.88 0) (unit 1)
+    (in_bom yes) (on_board yes) (fields_autoplaced)
+    (property "Reference" "H3" (id 0) (at 203.2 55.0453 0)
+      (effects (font (size 1.27 1.27)) (justify left))
+    )
+    (property "Value" "MountingHole" (id 1) (at 203.2 57.5822 0)
+      (effects (font (size 1.27 1.27)) (justify left))
+    )
+    (property "Footprint" "MountingHole:MountingHole_2.5mm_Pad_TopBottom" (id 2) (at 200.66 55.88 0)
+      (effects (font (size 1.27 1.27)) hide)
+    )
+    (property "Datasheet" "~" (id 3) (at 200.66 55.88 0)
+      (effects (font (size 1.27 1.27)) hide)
+    )
+  )
+  (symbol (lib_id "Mechanical:MountingHole") (at 200.66 68.58 0) (unit 1)
+    (in_bom yes) (on_board yes) (fields_autoplaced)
+    (property "Reference" "H4" (id 0) (at 203.2 67.7453 0)
+      (effects (font (size 1.27 1.27)) (justify left))
+    )
+    (property "Value" "MountingHole" (id 1) (at 203.2 70.2822 0)
+      (effects (font (size 1.27 1.27)) (justify left))
+    )
+    (property "Footprint" "MountingHole:MountingHole_2.5mm_Pad_TopBottom" (id 2) (at 200.66 68.58 0)
+      (effects (font (size 1.27 1.27)) hide)
+    )
+    (property "Datasheet" "~" (id 3) (at 200.66 68.58 0)
+      (effects (font (size 1.27 1.27)) hide)
+    )
   )
   (symbol (lib_id "power:+3V3") (at 248.92 99.06 0) (unit 1)
@@
     )
     (pin "1")
+  )
+  (symbol (lib_id "Mechanical:MountingHole") (at 175.26 68.58 0) (unit 1)
+    (in_bom yes) (on_board yes) (fields_autoplaced)
+    (property "Reference" "H2" (id 0) (at 177.8 67.7453 0)
+      (effects (font (size 1.27 1.27)) (justify left))
+    )
+    (property "Value" "MountingHole" (id 1) (at 177.8 70.2822 0)
+      (effects (font (size 1.27 1.27)) (justify left))
+    )
+    (property "Footprint" "MountingHole:MountingHole_2.5mm_Pad_TopBottom" (id 2) (at 175.26 68.58 0)
+      (effects (font (size 1.27 1.27)) hide)
+    )
+    (property "Datasheet" "~" (id 3) (at 175.26 68.58 0)
+      (effects (font (size 1.27 1.27)) hide)
+    )
   )
   (symbol (lib_id "power:GND") (at 241.3 35.56 0) (unit 1)
@@
     )
     (pin "1")
+  )
+  (symbol (lib_id "Mechanical:MountingHole") (at 175.26 55.88 0) (unit 1)
+    (in_bom yes) (on_board yes) (fields_autoplaced)
+    (property "Reference" "H1" (id 0) (at 177.8 55.0453 0)
+      (effects (font (size 1.27 1.27)) (justify left))
+    )
+    (property "Value" "MountingHole" (id 1) (at 177.8 57.5822 0)
+      (effects (font (size 1.27 1.27)) (justify left))
+    )
+    (property "Footprint" "MountingHole:MountingHole_2.5mm_Pad_TopBottom" (id 2) (at 175.26 55.88 0)
+      (effects (font (size 1.27 1.27)) hide)
+    )
+    (property "Datasheet" "~" (id 3) (at 175.26 55.88 0)
+      (effects (font (size 1.27 1.27)) hide)
+    )
   )
   (symbol (lib_id "power:+3V3") (at 198.12 25.4 0) (unit 1)
@@
   (symbol (lib_id "Regulator_Linear:LP5907MFX-3.3") (at 190.5 27.94 0) (unit 1)
     (in_bom yes) (on_board yes) (fields_autoplaced)
-    (property "Reference" "U?" (id 0) (at 190.5 19.1602 0))
+    (property "Reference" "U4" (id 0) (at 190.5 19.1602 0))
     (property "Value" "LP5907MFX-3.3" (id 1) (at 190.5 21.6971 0))
     (property "Footprint" "Package_TO_SOT_SMD:SOT-23-5" (id 2) (at 190.5 19.05 0)
@@
       (reference "#PWR0101") (unit 1) (value "GND") (footprint "")
     )
+    (path "/646574c8-b4b3-4708-bf3a-e9a7e40782e6"
+      (reference "H1") (unit 1) (value "MountingHole") (footprint "MountingHole:MountingHole_2.5mm_Pad_TopBottom")
+    )
+    (path "/35fd38cf-b64a-4f67-a191-ad442fca14a3"
+      (reference "H2") (unit 1) (value "MountingHole") (footprint "MountingHole:MountingHole_2.5mm_Pad_TopBottom")
+    )
+    (path "/2396f58f-ed26-4158-a0a4-a27558a55be9"
+      (reference "H3") (unit 1) (value "MountingHole") (footprint "MountingHole:MountingHole_2.5mm_Pad_TopBottom")
+    )
+    (path "/2d986ead-cd29-452d-91df-e51a3e7f33a9"
+      (reference "H4") (unit 1) (value "MountingHole") (footprint "MountingHole:MountingHole_2.5mm_Pad_TopBottom")
+    )
     (path "/2efaa1c5-361a-403e-a759-5892d61acb1d"
       (reference "J1") (unit 1) (value "Power") (footprint "Connector_Phoenix_MC:PhoenixContact_MC_1,5_2-G-3.5_1x02_P3.50mm_Horizontal")
@@
       (reference "U3") (unit 1) (value "ICM-20602") (footprint "Package_LGA:LGA-16_3x3mm_P0.5mm_LayoutBorder3x5y")
     )
+    (path "/c4e3f7f4-8d53-46fd-b919-c9ccc72b8301"
+      (reference "U4") (unit 1) (value "LP5907MFX-3.3") (footprint "Package_TO_SOT_SMD:SOT-23-5")
+    )
     (path "/9129be61-c293-426e-8253-da17ff12f65c"
       (reference "U5") (unit 1) (value "USB3341") (footprint "Package_DFN_QFN:QFN-24-1EP_4x4mm_P0.5mm_EP2.6x2.6mm")
@@
       (reference "U6") (unit 1) (value "TPD2EUSB30A") (footprint "Package_TO_SOT_SMD:Texas_DRT-3")
     )
-    (path "/c4e3f7f4-8d53-46fd-b919-c9ccc72b8301"
-      (reference "U?") (unit 1) (value "LP5907MFX-3.3") (footprint "Package_TO_SOT_SMD:SOT-23-5")
-    )
-  )
+  )
