File: Hardware Design/EVCU Jan 10/EVCU/EVCU.kicad_sch (KiCad schematic)
At the start: 60 parts, among them J1 Conn_01x06, J2 Conn_01x02, J3 APPS_Conn, J4 Micro_SD_Card, J5 DB9_Male, U1 BD33FC0WEFJ_E2, U10 EMIF06-MSD02N16, U11 ESDALC6V1W5, U3 STM32L4R9ZITx, U5 MPU-6500, U6 SN65HVD230, U7 LM358, U8 LM358, U9 ESDCAN24-2BLY, X1 ECS-2520MV-160-CN-TR

Commit message: .
Connections:
- net +3V3: now also C29.2; no longer C29.1
- net FILTER_CS: now also U10.13 (DAT3_EX); no longer U10.4 (DAT3_In)
- net GND: now also C29.1; no longer C29.2
- net MISO: now also U10.7 (DAT0_In); no longer U10.10 (DAT0_Ex)
- net MOSI: now also U10.5 (CMD_In); no longer U10.12 (CMD_Ex)
- net SCK: now also U10.6 (CLK_In); no longer U10.11 (CLK_Ex)
- net SD_CS: now also U10.4 (DAT3_In); no longer U10.13 (DAT3_EX)
- net at J4.1 (DAT2): now also U10.14 (DAT2_Ex)
- net FILTER_DAT1: now reaches J4.8 (DAT1)
- net FILTER_DAT1: now also U10.9 (DAT1_Ex)
- net FILTER_MISO renamed FILTER_DAT0
- net FILTER_DAT0: now also U10.10 (DAT0_Ex); no longer U10.7 (DAT0_In)
- net FILTER_MOSI renamed FILTER_CMD
- net FILTER_CMD: now also U10.12 (CMD_Ex); no longer U10.5 (CMD_In)
- net FILTER_SCK renamed FILTER_CLK
- net FILTER_CLK: now also U10.11 (CLK_Ex); no longer U10.6 (CLK_In)
- no-connect marks 119 -> 115
